File: Electronique/Asservissement_Shield/Asservissement_Shield.kicad_pcb (KiCad board)
At the start: 2 copper layers, 4 parts, among them J1 Hall_Sensor, J2 Windings, J3 Hall_Sensor, J4 Windings

Commit message: routage
Parts:
- added C1: 100n, Capacitor_SMD:C_0805_2012Metric_Pad1.15x1.40mm_HandSolder, F.Cu at (119.0, 35.8)
- added C10: 10n, Capacitor_SMD:C_0805_2012Metric_Pad1.15x1.40mm_HandSolder, F.Cu at (124.8, 73.6)
- added C11: 5.6n, Capacitor_SMD:C_0805_2012Metric_Pad1.15x1.40mm_HandSolder, F.Cu at (105.0, 90.4)
- added C12: 1n, Capacitor_SMD:C_0805_2012Metric_Pad1.15x1.40mm_HandSolder, B.Cu at (116.2, 92.0)
- added C13: 10n, Capacitor_SMD:C_0805_2012Metric_Pad1.15x1.40mm_HandSolder, B.Cu at (114.2, 69.4)
- added C14: 220n, Capacitor_SMD:C_1206_3216Metric_Pad1.42x1.75mm_HandSolder, F.Cu at (120.0, 72.8)
- added C2: 100n, Capacitor_SMD:C_0805_2012Metric_Pad1.15x1.40mm_HandSolder, F.Cu at (110.0, 44.0)
- added C3: 1n, Capacitor_SMD:C_0805_2012Metric_Pad1.15x1.40mm_HandSolder, F.Cu at (85.0, 41.7)
- added C4: 10n, Capacitor_SMD:C_0805_2012Metric_Pad1.15x1.40mm_HandSolder, F.Cu at (78.3, 45.5)
- added C5: 5.6n, Capacitor_SMD:C_0805_2012Metric_Pad1.15x1.40mm_HandSolder, F.Cu at (80.3, 42.1)
- added C6: 1n, Capacitor_SMD:C_0805_2012Metric_Pad1.15x1.40mm_HandSolder, F.Cu at (80.3, 39.1)
- added C7: 10n, Capacitor_SMD:C_0805_2012Metric_Pad1.15x1.40mm_HandSolder, F.Cu at (85.8, 38.8)
- added C8: 220n, Capacitor_SMD:C_1206_3216Metric_Pad1.42x1.75mm_HandSolder, F.Cu at (54.0, 53.1)
- added C9: 1n, Capacitor_SMD:C_0805_2012Metric_Pad1.15x1.40mm_HandSolder, B.Cu at (109.8, 92.0)
- added D1: 1N4148, Diode_SMD:D_SOD-123F, F.Cu at (80.7, 36.0)
- added D2: 1N4148, Diode_SMD:D_SOD-123F, F.Cu at (59.7, 53.1)
- added D3: 1N4148, Diode_SMD:D_SOD-123F, B.Cu at (115.6, 73.4)
- added D4: 1N4148, Diode_SMD:D_SOD-123F, B.Cu at (118.6, 73.4)
- added P1: encoder_2, Connector_Molex:Molex_KK-254_AE-6410-04A_1x04_P2.54mm_Vertical, F.Cu at (97.8, 38.3)
- added P2: encoder_2, Connector_Molex:Molex_KK-254_AE-6410-04A_1x04_P2.54mm_Vertical, F.Cu at (97.8, 46.1)
- added R1: 1k, Resistor_SMD:R_0805_2012Metric_Pad1.15x1.40mm_HandSolder, F.Cu at (83.0, 53.9)
- added R10: 0, Resistor_SMD:R_0805_2012Metric_Pad1.15x1.40mm_HandSolder, F.Cu at (78.3, 48.4)
- added R11: 0, Resistor_SMD:R_0805_2012Metric_Pad1.15x1.40mm_HandSolder, F.Cu at (85.8, 35.8)
- added R12: 1k, Resistor_SMD:R_0805_2012Metric_Pad1.15x1.40mm_HandSolder, F.Cu at (101.6, 91.2)
- added R13: 100k, Resistor_SMD:R_0805_2012Metric_Pad1.15x1.40mm_HandSolder, F.Cu at (105.0, 86.2)
- added R14: 35k, Resistor_SMD:R_0805_2012Metric_Pad1.15x1.40mm_HandSolder, B.Cu at (112.2, 92.0)
- added R15: 1k2, Resistor_SMD:R_0805_2012Metric_Pad1.15x1.40mm_HandSolder, F.Cu at (122.4, 73.6)
- added R16: 220, Resistor_SMD:R_0805_2012Metric_Pad1.15x1.40mm_HandSolder, F.Cu at (127.2, 73.6)
- added R17: 47k, Resistor_SMD:R_0805_2012Metric_Pad1.15x1.40mm_HandSolder, B.Cu at (118.6, 92.0)
- added R18: 100, Resistor_SMD:R_0805_2012Metric_Pad1.15x1.40mm_HandSolder, B.Cu at (112.6, 73.4)
- added R19: 0.3, Resistor_SMD:R_1206_3216Metric_Pad1.42x1.75mm_HandSolder, F.Cu at (109.4, 92.4)
- added R2: 100k, Resistor_SMD:R_0805_2012Metric_Pad1.15x1.40mm_HandSolder, F.Cu at (87.8, 47.6)
- added R20: 0, Resistor_SMD:R_0805_2012Metric_Pad1.15x1.40mm_HandSolder, F.Cu at (105.0, 63.4)
- added R21: 0, Resistor_SMD:R_0805_2012Metric_Pad1.15x1.40mm_HandSolder, F.Cu at (107.0, 63.4)
- added R22: 0, Resistor_SMD:R_0805_2012Metric_Pad1.15x1.40mm_HandSolder, F.Cu at (103.0, 63.4)
- added R3: 35k, Resistor_SMD:R_0805_2012Metric_Pad1.15x1.40mm_HandSolder, F.Cu at (83.0, 51.0)
- added R4: 1k2, Resistor_SMD:R_0805_2012Metric_Pad1.15x1.40mm_HandSolder, F.Cu at (78.3, 54.3)
- added R5: 220, Resistor_SMD:R_0805_2012Metric_Pad1.15x1.40mm_HandSolder, F.Cu at (87.8, 44.6)
- added R6: 47k, Resistor_SMD:R_0805_2012Metric_Pad1.15x1.40mm_HandSolder, F.Cu at (83.0, 48.0)
- added R7: 100, Resistor_SMD:R_0805_2012Metric_Pad1.15x1.40mm_HandSolder, F.Cu at (89.8, 41.7)
- added R8: 0.3, Resistor_SMD:R_1206_3216Metric_Pad1.42x1.75mm_HandSolder, F.Cu at (78.3, 51.4)
- added R9: 0, Resistor_SMD:R_0805_2012Metric_Pad1.15x1.40mm_HandSolder, F.Cu at (83.0, 45.0)
- added U1: TXS0108EPW, Package_SO:TSSOP-20_4.4x6.5mm_P0.65mm, F.Cu at (112.2, 38.4)
- added U2: L6235PD, Package_SO:SOIC-24W_7.5x15.4mm_P1.27mm, F.Cu at (57.5, 42.9)
- added U3: L6235PD, Package_SO:SOIC-24W_7.5x15.4mm_P1.27mm, F.Cu at (115.4, 82.8)
- moved J1 138.1 mm to (66.9, 36.7)
- moved J4 106.5 mm to (127.2, 85.4), turned to 90 degrees
- moved J3 94.8 mm to (109.0, 72.8), turned to 180 degrees
- moved J2 82.5 mm to (137.2, 41.2), turned to 90 degrees
Connections:
- J1 pad 2: (no net) -> /MotorA/Hall_Sensor2
- J1 pad 3: (no net) -> /MotorA/Hall_Sensor1
- J1 pad 4: (no net) -> /MotorA/Hall_Sensor3
- J2 pad 1: (no net) -> /MotorA/Motor_Winding1
- J2 pad 2: (no net) -> /MotorA/Motor_Winding2
- J2 pad 3: (no net) -> /MotorA/Motor_Winding3
- J3 pad 2: (no net) -> /MotorB/Hall_Sensor2
- J3 pad 3: (no net) -> /MotorB/Hall_Sensor1
- J3 pad 4: (no net) -> /MotorB/Hall_Sensor3
- J4 pad 1: (no net) -> /MotorB/Motor_Winding1
- J4 pad 2: (no net) -> /MotorB/Motor_Winding2
- J4 pad 3: (no net) -> /MotorB/Motor_Winding3
Routing:
- net (no net): track 0.00 -> 42.6 mm, vias 0 -> 1
- net /Diagnostic_1: track 0.00 -> 34.8 mm
- net /MotorB/Hall_Sensor1: track 0.00 -> 25.7 mm
- net /Tachometer_1: track 0.00 -> 21.1 mm
- net /MotorB/Motor_Winding2: track 0.00 -> 17.8 mm
- net VCC: track 0.00 -> 17.7 mm, vias 0 -> 1
- net /MotorB/Hall_Sensor3: track 0.00 -> 16.2 mm
- net /MotorB/Motor_Winding1: track 0.00 -> 15.5 mm
- net /MotorB/Hall_Sensor2: track 0.00 -> 14.8 mm
- net /MotorB/Motor_Winding3: track 0.00 -> 10.5 mm
- net Net-(C10-Pad1): track 0.00 -> 8.28 mm
- net Net-(C14-Pad1): track 0.00 -> 6.14 mm, vias 0 -> 1
- net Net-(C9-Pad1): track 0.00 -> 5.89 mm, vias 0 -> 1
- net Net-(C12-Pad1): track 0.00 -> 5.87 mm, vias 0 -> 1
- net Net-(C13-Pad1): track 0.00 -> 5.76 mm
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
Commit message: oops
Parts:
- R19: moved to B.Cu
- moved C13 32.3 mm to (138.0, 91.2), turned to 90 degrees
- moved R22 32.2 mm to (133.0, 75.2), turned to 180 degrees
- moved R16 31.3 mm to (133.8, 104.2), turned to 0 degrees
- moved R20 31.2 mm to (133.0, 77.2), turned to 180 degrees
- moved R21 30.4 mm to (133.0, 79.2), turned to 180 degrees
- moved C10 29.6 mm to (133.8, 101.8), turned to 0 degrees
- moved C14 28.3 mm to (134.6, 97.0), turned to 0 degrees
- moved R15 28.2 mm to (133.8, 99.4), turned to 180 degrees
- moved D4 27.0 mm to (134.0, 95.6), turned to 0 degrees
- moved R18 26.8 mm to (134.0, 89.6), turned to 180 degrees
- moved D3 26.6 mm to (134.0, 92.6), turned to 180 degrees
- moved J3 21.2 mm to (128.6, 81.0)
- moved J4 19.5 mm to (122.0, 104.2), turned to 0 degrees
- moved C11 13.6 mm to (115.8, 82.2), turned to 180 degrees
- moved U3 13.3 mm to (124.6, 92.4), turned to 0 degrees
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Routing:
- net GND: track 2.54 -> 40.6 mm, vias 0 -> 3
- net /Diagnostic_1: track 34.8 -> 6.81 mm
- net /MotorB/Hall_Sensor3: track 16.2 -> 36.6 mm
- net (no net): track 42.6 -> 28.2 mm, vias 1 -> 2
- net Net-(R19-Pad2): track 0.00 -> 13.2 mm, vias 0 -> 2
- net /Tachometer_1: track 21.1 -> 8.15 mm
- net /MotorB/Hall_Sensor1: track 25.7 -> 16.8 mm
- net Net-(C12-Pad1): track 5.87 -> 10.9 mm
- net /MotorB/Hall_Sensor2: track 14.8 -> 14.0 mm
- added copper zone on B.Cu, net GND
- added copper zone on F.Cu, net GND
